Commit message: new messages & custom KUKA functions

File: iiwa_description/urdf/MRobot_Gazebo.urdf (robot description, URDF)
Before this commit: robot m_robot, 31 links, 30 joints
Links:
- added link ceiling; collision box size=10.0 10.0 0.001
Joints:
- added joint ceiling_base: type fixed, parent base_link, child ceiling, origin xyz=0.0 0.0 2.2 rpy=0 0 0
- joint m_robot_joint_2: limit lower=-2.0943951023931953 upper=2.0943951023931953 effort=300 velocity=10 -> lower=-2.00713 upper=2.00713 effort=300 velocity=10
- joint m_robot_joint_4: limit lower=-2.0943951023931953 upper=2.0943951023931953 effort=300 velocity=10 -> lower=-2.00713 upper=2.00713 effort=300 velocity=10
- joint m_robot_joint_6: limit lower=-2.0943951023931953 upper=2.0943951023931953 effort=300 velocity=10 -> lower=-2.00713 upper=1.91986 effort=300 velocity=10
- joint m_robot_linear_drive_dof1_dof2_joint: limit lower=-1.4 upper=-0.15 effort=1 velocity=0.95 -> lower=-1.571 upper=0.0 effort=1 velocity=0.95
- joint m_robot_linear_drive_guiderail_sledge_joint: limit lower=0.0 upper=0.33 effort=1 velocity=0.95 -> lower=0.0 upper=0.25 effort=1 velocity=0.95; origin xyz=0 0.08 0.0413 rpy=0 0 0 -> xyz=0 0.15 0.0413 rpy=0 0 0
- joint m_robot_linear_drive_link_ee_Soft_RG6_joint: origin xyz=-0.0035 0.4 0.0 rpy=0 1.571 -1.571 -> xyz=-0.0035 0.4 -0.005 rpy=0 1.571 -1.571
- joint m_robot_support_structure_m_robot_joint: origin xyz=0 -1.05 0.51 rpy=0 0 1.5707963267948966 -> xyz=0 -1.05 0.885 rpy=0 0 1.5707963267948966

Commit message: nasekomo

File: iiwa_description/urdf/MRobot_Gazebo.urdf (robot description, URDF)
Before this commit: robot m_robot, 32 links, 31 joints
Links:
- removed link ceiling
- removed link zed2i_baro_link
- removed link zed2i_base_link
- removed link zed2i_camera_center
- removed link zed2i_left_camera_frame
- removed link zed2i_left_camera_optical_frame
- removed link zed2i_mag_link
- removed link zed2i_right_camera_frame
- removed link zed2i_right_camera_optical_frame
- removed link zed2i_temp_left_link
- removed link zed2i_temp_right_link
- added link artificial_ceiling; collision box size=10.0 10.0 0.001
- added link realsense_base_link, mass 0.1; collision mesh filename=package://iiwa_description/meshes/RealSense D435/d435.dae; visual mesh filename=package://iiwa_description/meshes/RealSense D435/d435.dae
- link m_robot_linear_drive_dof1: geometry collision mesh filename=package://iiwa_description/meshes/Linear Drive Sept2023/2 D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; visual mesh filename=package://iiwa_description/meshes/Linear Drive Sept2023/2 D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
- link m_robot_linear_drive_dof2: geometry collision mesh filename=package://iiwa_description/meshes/Linear Drive Sept2023/3DO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; visual mesh filename=package://iiwa_description/meshes/Linear Drive Sept2023/3DO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
- link m_robot_linear_drive_guiderail: geometry collision mesh filename=package://iiwa_description/meshes/Linear Drive Sept2023/Gui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; visual mesh filename=package://iiwa_description/meshes/Linear Drive Sept2023/Gui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
- link m_robot_linear_drive_sledge: geometry collision mesh filename=package://iiwa_description/meshes/Linear Drive Sept2023/Sle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; visual mesh filename=package://iiwa_description/meshes/Linear Drive Sept2023/Sle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
Joints:
- removed joint ceiling_base
- removed joint zed2i_baro_joint
- removed joint zed2i_base_joint
- removed joint zed2i_camera_center_joint
- removed joint zed2i_left_camera_joint
- removed joint zed2i_left_camera_optical_joint
- removed joint zed2i_mag_joint
- removed joint zed2i_right_camera_joint
- removed joint zed2i_right_camera_optical_joint
- removed joint zed2i_temp_left_joint
- removed joint zed2i_temp_right_joint
- added joint artificial_ceiling_to_base: type fixed, parent base_link, child artificial_ceiling, origin xyz=0.0 0.0 2.2 rpy=0 0 0
- added joint realsense_base_joint: type fixed, parent Soft_RG6_finger_2, child realsense_base_link, origin xyz=0 0.05 0.1 rpy=0 0 -1.57
- joint m_robot_linear_drive_dof1_dof2_joint: origin xyz=-0.02 0.005 0.074 rpy=0 0 0 -> xyz=0 0 -0.071 rpy=0 0 0
- joint m_robot_linear_drive_guiderail_sledge_joint: limit lower=0.0 upper=0.25 effort=1 velocity=0.95 -> lower=0.0 upper=0.33 effort=1 velocity=0.3; origin xyz=0 0.15 0.0413 rpy=0 0 0 -> xyz=0 -0.12 -0.022 rpy=0 0 3.14159
- joint m_robot_linear_drive_joint_ee: origin xyz=0.02 -0.32 0.08 rpy=0 0 0 -> xyz=0 0.32 -0.0625 rpy=0 0 0
- joint m_robot_linear_drive_link_ee_Soft_RG6_joint: origin xyz=-0.0035 0.4 -0.005 rpy=0 1.571 -1.571 -> xyz=0 -0.385 0 rpy=3.14159 1.571 -1.571
- joint m_robot_linear_drive_sledge_dof1_joint: origin xyz=0 0 0 rpy=0 0 3.1415 -> xyz=0 0 -0.015 rpy=0 0 0
- joint m_robot_link_ee_m_robot_joint_ee: origin xyz=0.08 0 0.08 rpy=0 0 1.5707963267948966 -> xyz=0.07 0 0.043 rpy=3.14159 0 1.5707963267948966
- joint m_robot_support_structure_m_robot_joint: origin xyz=0 -1.05 0.885 rpy=0 0 1.5707963267948966 -> xyz=0 -1.05 0.885 rpy=0 0 0

Commit message: changes

File: iiwa_description/urdf/MRobot_Gazebo.urdf (robot description, URDF)
Before this commit: robot m_robot, 23 links, 22 joints
Joints:
- joint m_robot_joint_1: limit lower=-2.9670597283903604 upper=2.9670597283903604 effort=300 velocity=10 -> lower=-2.9321531433504737 upper=2.9321531433504737 effort=300 velocity=10
- joint m_robot_joint_2: limit lower=-2.00713 upper=2.00713 effort=300 velocity=10 -> lower=-2.0594885173533086 upper=2.0594885173533086 effort=300 velocity=10
- joint m_robot_joint_3: limit lower=-2.9670597283903604 upper=2.9670597283903604 effort=300 velocity=10 -> lower=-2.9321531433504737 upper=2.9321531433504737 effort=300 velocity=10
- joint m_robot_joint_4: limit lower=-2.00713 upper=2.00713 effort=300 velocity=10 -> lower=-2.0594885173533086 upper=2.0594885173533086 effort=300 velocity=10
- joint m_robot_joint_5: limit lower=-2.9670597283903604 upper=2.9670597283903604 effort=300 velocity=10 -> lower=-1.7453292519943295 upper=1.7453292519943295 effort=300 velocity=10
- joint m_robot_joint_6: limit lower=-2.00713 upper=1.91986 effort=300 velocity=10 -> lower=-2.0094885173533086 upper=2.0094885173533086 effort=300 velocity=10
- joint m_robot_support_structure_m_robot_joint: origin xyz=0 -1.05 0.885 rpy=0 0 0 -> xyz=0 -1.05 0.885 rpy=0 0 1.571

Commit message: final changes before entomotech

File: iiwa_description/urdf/MRobot_Gazebo.urdf (robot description, URDF)
Before this commit: robot m_robot, 23 links, 22 joints
Links:
- added link certh_horizontal_link, mass 0.1; collision mesh filename=package://iiwa_description/meshes/certh_camera/CERTH_Camera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; visual mesh filename=package://iiwa_description/meshes/certh_camera/CERTH_Camera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
- added link certh_vertical_link, mass 0.1; collision mesh filename=package://iiwa_description/meshes/certh_camera/CERTH_Camera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; visual mesh filename=package://iiwa_description/meshes/certh_camera/CERTH_Camera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
Joints:
- added joint certh_horizontal_joint: type fixed, parent m_robot_linear_drive_guiderail, child certh_horizontal_link, origin xyz=-0.0325 -0.19 0 rpy=0 3.1415 3.1415
- added joint certh_vertical_joint: type fixed, parent certh_horizontal_link, child certh_vertical_link, origin xyz=0.0325 0.3725 0.12 rpy=3.1415 0 1.571
- joint artificial_ceiling_to_base: origin xyz=0.0 0.0 2.2 rpy=0 0 0 -> xyz=0.0 0.0 2. rpy=0 0 0
- joint m_robot_linear_drive_dof1_dof2_joint: limit lower=-1.571 upper=0.0 effort=1 velocity=0.95 -> lower=-1.571 upper=0.0 effort=1 velocity=1.571
- joint m_robot_linear_drive_sledge_dof1_joint: limit lower=-1.571 upper=1.571 effort=1 velocity=0.95 -> lower=-1.571 upper=1.571 effort=1 velocity=1.571
